Commit message: adding urdf, works with motoman driver install (not included in this repo). works in ros1

File: ros2_ws/src/snp_support/urdf/workcell.xacro (robot description, xacro)
@@ -1,5 +1,7 @@
 <?xml version="1.0" ?>
-<robot name="snp_workcell" xmlns:xacro="http://ros.org/wiki/xacro">
-  <xacro:include filename="$(find snp_support)/urdf/mh180_120.xacro"/>
+<robot name="motoman_hc10" xmlns:xacro="http://ros.org/wiki/xacro">
+  <xacro:include filename="$(find motoman_hc10_support)/urdf/hc10_macro.xacro" />
+  <xacro:motoman_hc10 prefix=""/>
+  <!-- link list -->
   <material name="light_gray">
     <color rgba="0.7 0.7 0.7 1"/>
@@ -11,10 +13,10 @@
     <visual>
       <geometry>
-        <mesh filename="package://snp_support/meshes/pushcorp/pushcorp_base.dae"/>
+        <mesh filename="package://inspection_cell_support/meshes/pushcorp/pushcorp_base.dae"/>
       </geometry>
     </visual>
     <collision>
       <geometry>
-        <mesh filename="package://snp_support/meshes/pushcorp/pushcorp_base.dae"/>
+        <mesh filename="package://inspection_cell_support/meshes/pushcorp/pushcorp_base.dae"/>
       </geometry>
     </collision>
@@ -22,26 +24,41 @@
   <link name="pushcorp_compliance">
     <visual>
-      <origin xyz="0 0.059 0" rpy="${pi} 0 0"/>
+      <origin xyz="0.05 -0.05 0.05" rpy="0 ${radians(90)} 0"/>
       <geometry>
-        <mesh filename="package://snp_support/meshes/pushcorp/pushcorp_spindle.dae"/>
+        <mesh filename="package://inspection_cell_support/meshes/collision_demo/rps100.STL"/>
       </geometry>
       <material name="light_gray"/>
     </visual>
     <collision>
-      <origin xyz="0 0.059 0" rpy="${pi} 0 0"/>
+      <origin xyz="0.05 -0.05 0.05" rpy="0 ${radians(90)} 0"/>
       <geometry>
-        <mesh filename="package://snp_support/meshes/pushcorp/pushcorp_spindle.dae"/>
+        <mesh filename="package://inspection_cell_support/meshes/collision_demo/rps100.STL"/>
       </geometry>
     </collision>
   </link>
+<link name="pushcorp_bracket">
+  <visual>
+    <origin xyz="0.165 -0.035 -0.175" rpy="0 0 ${radians(90)}"/>
+    <geometry>
+      <mesh filename="package://inspection_cell_support/meshes/collision_demo/camera mount as part.STL"/>
+    </geometry>
+    <material name="light_gray"/>
+  </visual>
+  <collision>
+    <origin xyz="0 0 0" rpy="0 0 ${radians(90)}"/>
+    <geometry>
+      <mesh filename="package://inspection_cell_support/meshes/collision_demo/camera mount as part.STL"/>
+    </geometry>
+  </collision>
+</link>
   <link name="camera_link"/>
-  <link name="target_base_link">
+  <!-- link name="target_base_link">
     <visual>
       <origin xyz="0.37565 0.2809875 0" rpy="${pi/2} 0 ${pi}"/>
       <geometry>
-        <mesh filename="package://snp_support/meshes/rosWorldCalib.dae"/>
+        <mesh filename="package://inspection_cell_support/meshes/rosWorldCalib.dae"/>
       </geometry>
     </visual>
-  </link>
+  </link-->
   <joint name="tool0_to_pushcorp_base" type="fixed">
     <parent link="tool0"/>
@@ -52,15 +69,15 @@
     <parent link="tool0"/>
     <child link="camera_link"/>
-    <origin xyz="0 0 0" rpy="0 0 0"/>
+    <origin xyz="0.175 0 0" rpy="0 0 0"/>
     <axis xyz="0 0 0"/>
   </joint>
-  <joint name="world_to_target_joint" type="fixed">
+  <!-- joint name="world_to_target_joint" type="fixed">
     <parent link="floor"/>
     <child link="target_base_link"/>
     <origin xyz="0.555 0.061 0.126" rpy="0.004 -0.004 -1.628"/>
     <axis xyz="0 0 0"/>
-  </joint>
+  </joint-->
   <link name="camera_color_optical_frame"/>
-  <link name="target_cal_frame"/>
+  <!--link name="target_cal_frame"/-->
   <joint name="camera_cal_joint" type="fixed">
     <parent link="camera_link"/>
@@ -68,148 +85,60 @@
     <origin xyz="0.085549560652492 -0.1732631672558103 0.1329373703855808" wxyz="0.5118596229748543 -0.5074314040915237 0.4900425218487801 -0.4902768843111336"/>
   </joint>
-  <joint name="target_cal_joint" type="fixed">
+  <!--joint name="target_cal_joint" type="fixed">
     <parent link="floor"/>
     <child link="target_cal_frame"/>
     <origin xyz="0.555641489380775 0.05956001933889868 0.1229851433910979" wxyz="0.6869783604862724 -0.001114251051880176 -0.003909064875724348 -0.7266665052690842"/>
-  </joint>
+  </joint-->
   <!-- TODO do we care about effort and velocity limits?-->
-  <joint name="pushcorp_actuator" type="prismatic">
+  <joint name="pushcorp_actuator" type="fixed">
     <parent link="pushcorp_base"/>
     <child link="pushcorp_compliance"/>
     <origin xyz="0 0 0" rpy="0 0 0"/>
-    <axis xyz="-1 0 0"/>
+    <axis xyz="0 1 0"/>
     <limit upper="0.01778" lower="-0.01778" effort="0" velocity="0"/>
   </joint>
-  <xacro:property name="platform_height" value="${5*0.0254}"/>
-  <xacro:property name="robot_mount_height" value="${19.6*0.0254}"/>
-  <xacro:property name="robot_mount_width" value="${28.5*0.0254}"/>
-  <xacro:property name="pushcorp_box_height" value="${30*0.0254}"/>
-  <xacro:property name="pushcorp_box_width" value="${17*0.0254}"/>
-  <xacro:property name="pushcorp_box_length" value="${28*0.0254}"/>
-  <xacro:property name="control_boxes_height" value="${60*0.0254}"/>
-  <xacro:property name="control_boxes_width" value="${38*0.0254}"/>
-  <xacro:property name="control_boxes_length" value="${130*0.0254}"/>
-  <xacro:property name="table_height" value="${33.875*0.0254}"/>
-  <xacro:property name="table_width" value="${48*0.0254}"/>
-  <xacro:property name="table_length" value="${30*0.0254}"/>
+<!-- joint name="pushcorp_actuator" type="fixed">
+  <parent link="pushcorp_base"/>
+  <child link="pushcorp_compliance"/>
+  <origin xyz="0 0 0" rpy="0 0 0"/>
+  <axis xyz="0 1 0"/>
+  <limit upper="0.01778" lower="-0.01778" effort="0" velocity="0"/>
+</joint-->
+<joint name="pushcorp_bracket" type="fixed">
+  <parent link="pushcorp_base"/>
+  <child link="pushcorp_bracket"/>
+  <origin xyz="0 0 0" rpy="0 0 0"/>
+</joint>
   <link name="floor"/>
-  <link name="platform">
+  <link name="robot_mount">
     <visual>
+      <origin xyz="0.61 0 -0.75" rpy="0 0 0"/> <!-- origin xyz="x= -z,  -0.04 -0.06" rpy="0 0 0"/-->
       <geometry>
-        <box size="${96*0.0254} ${72*0.0254} ${platform_height}"/>
+        <mesh filename="package://inspection_cell_support/meshes/collision_demo/Steel Table 4 ft x 6ft.STL"/>
       </geometry>
       <material name="dark_gray"/>
     </visual>
     <collision>
+    <origin xyz="0.61 0 -0.35" rpy="0 0 0"/>
       <geometry>
-        <box size="${96*0.0254} ${72*0.0254} ${platform_height}"/>
+        <box size="2 1 0.7"/>
       </geometry>
     </collision>
   </link>
-  <link name="robot_mount">
-    <visual>
-      <geometry>
-        <box size="${robot_mount_width} ${robot_mount_width} ${robot_mount_height}"/>
-      </geometry>
-      <material name="dark_gray"/>
-    </visual>
-    <collision>
-      <geometry>
-        <box size="${robot_mount_width} ${robot_mount_width} ${robot_mount_height}"/>
-      </geometry>
-    </collision>
-  </link>
-  <link name="pushcorp_box_support_1">
-    <visual>
-      <geometry>
-        <box size="${1.5*0.0254} ${1.5*0.0254} ${40.5*0.0254}" />
-      </geometry>
-      <material name="dark_gray"/>
-    </visual>
-    <collision>
-      <geometry>
-        <box size="${1.5*0.0254} ${1.5*0.0254} ${40.5*0.0254}" />
-      </geometry>
-    </collision>
-  </link>
-  <link name="pushcorp_box_support_2">
-    <visual>
-      <geometry>
-        <box size="${1.5*0.0254} ${1.5*0.0254} ${40.5*0.0254}" />
-      </geometry>
-      <material name="dark_gray"/>
-    </visual>
-    <collision>
-      <geometry>
-        <box size="${1.5*0.0254} ${1.5*0.0254} ${40.5*0.0254}" />
-      </geometry>
-    </collision>
-  </link>
-  <link name="pushcorp_box">
-    <visual>
-      <geometry>
-        <box size="${pushcorp_box_length} ${pushcorp_box_width} ${pushcorp_box_height}"/>
-      </geometry>
-      <material name="light_gray"/>
-    </visual>
-    <collision>
-      <geometry>
-        <box size="${pushcorp_box_length} ${pushcorp_box_width} ${pushcorp_box_height}"/>
-      </geometry>
-    </collision>
-  </link>
-  <link name="control_boxes">
-   <visual>
-      <geometry>
-        <box size="${control_boxes_length} ${control_boxes_width} ${control_boxes_height}"/>
-      </geometry>
-      <material name="light_gray"/>
-    </visual>
-    <collision>
-      <geometry>
-        <box size="${control_boxes_length} ${control_boxes_width} ${control_boxes_height}"/>
-      </geometry>
-    </collision>
-  </link>
-  <link name="buffy_tcp"/>
-  <joint name="buffy_tcp_joint" type="fixed">
+  <link name="sand_tcp"/>
+  <joint name="sand_tcp_joint" type="fixed">
     <parent link="tool0"/>
-    <child link="buffy_tcp"/>
-    <origin xyz="0.292 0 0.19" rpy="0 -${pi/2} 0"/>
+    <child link="sand_tcp"/>
+    <origin xyz="0.2 0 0.045" rpy="0 0 0"/>
   </joint>
-  <joint name="floor_to_platform" type="fixed">
+  <joint name="floor_to_robot_mount" type="fixed">
     <parent link="floor"/>
-    <child link="platform"/>
-    <origin xyz="0 0 ${platform_height/2}" rpy="0 0 0"/>
-  </joint>
-  <joint name="platform_to_mount" type="fixed">
-    <parent link="platform"/>
     <child link="robot_mount"/>
-    <origin xyz="0 0 ${platform_height/2 + robot_mount_height/2}" rpy="0 0 0"/>
-  </joint>
-  <joint name="floor_to_control_boxes" type="fixed">
-    <parent link="floor"/>
-    <child link="control_boxes"/>
-    <origin xyz="${4*0.0254 + control_boxes_length/2} -${56*0.0254 + control_boxes_width/2} ${control_boxes_height/2}" rpy="0 0 0"/>
+    <origin xyz="0 0 0" rpy="0 0 0"/>
   </joint>
   <joint name="mount_to_base" type="fixed">
     <parent link="robot_mount"/>
     <child link="base_link"/>
-    <origin xyz="0 0 ${robot_mount_height/2}" rpy="0 0 0"/>
-  </joint>
-  <joint name="floor_to_pushcorp_support_1" type="fixed">
-    <parent link="floor"/>
-    <child link="pushcorp_box_support_1"/>
-    <origin xyz="-${robot_mount_width/2 + 2.75*0.0254} ${robot_mount_width/2 + 16.25*0.0254} ${20.25*0.0254+platform_height}" rpy="0 0 0"/>
-  </joint>
-  <joint name="floor_to_pushcorp_support_2" type="fixed">
-    <parent link="floor"/>
-    <child link="pushcorp_box_support_2"/>
-    <origin xyz="-${robot_mount_width/2 + 1.25*0.0254 + pushcorp_box_length} ${robot_mount_width/2 + 16.25*0.0254} ${20.25*0.0254+platform_height}" rpy="0 0 0"/>
-  </joint>
-  <joint name="floor_to_pushcorp_box" type="fixed">
-    <parent link="floor"/>
-    <child link="pushcorp_box"/>
-    <origin xyz="-${robot_mount_width/2 + 2*0.0254 + pushcorp_box_length/2} ${robot_mount_width/2 + 17*0.0254 + pushcorp_box_width/2} ${14*0.0254 + pushcorp_box_height/2}" rpy="0 0 0"/>
+    <origin xyz="0 0 0" rpy="0 0 0"/>
   </joint>
 </robot>
